Commit message: add neor_mini line-tracking ros node

File: mini_sim18_ws/src/neor_mini/urdf/neor_mini_gazebo_sensors.urdf (robot description, URDF)
Before this commit: robot neor_mini, 13 links, 12 joints
Links:
- link base_link: geometry collision mesh filename=package://neor_mini/meshes/base_link.STL; visual mesh filename=package://neor_mini/meshes/base_link.STL
